Commit message: add gpd cloud

File: src/kinova-ros/kinova_description/urdf/j2s7s300.xacro (robot description, xacro)
@@ -44,5 +44,5 @@
     <xacro:property name="joint_base_axis_xyz" value="0 0 0" />
     <xacro:property name="joint_base_origin_xyz" value="0 0 0" />
-    <xacro:property name="joint_base_origin_rpy" value="0 0 0" />
+    <xacro:property name="joint_base_origin_rpy" value="0 0 -1.57" />
     <xacro:property name="joint_1" value="joint_1" />
     <xacro:property name="joint_1_type" value="continuous" />

File: src/kinova-ros/kinova_description/urdf/j2s7s300_standalone.xacro (robot description, xacro)
@@ -18,65 +18,8 @@
   <!-- for gazebo -->
   <link name="world"/>
-  <!-- <model name='unit_box'>
-    <pose>0.0508 -0.231174 0.5 0 -0 0</pose>
-    <link name='box_link'>
-      <inertial>
-        <mass>1</mass>
-        <inertia>
-          <ixx>0.166667</ixx>
-          <ixy>0</ixy>
-          <ixz>0</ixz>
-          <iyy>0.166667</iyy>
-          <iyz>0</iyz>
-          <izz>0.166667</izz>
-        </inertia>
-        <pose>0 0 0 0 -0 0</pose>
-      </inertial>
-      <collision name='collision'>
-        <geometry>
-          <box>
-            <size>1 1 0.4</size>
-          </box>
-        </geometry>
-        <max_contacts>10</max_contacts>
-        <surface>
-          <contact>
-            <ode/>
-          </contact>
-          <bounce/>
-          <friction>
-            <torsional>
-              <ode/>
-            </torsional>
-            <ode/>
-          </friction>
-        </surface>
-      </collision>
-      <visual name='visual'>
-        <geometry>
-          <box>
-            <size>1 1 0.999998</size>
-          </box>
-        </geometry>
-        <material>
-          <script>
-            <name>Gazebo/Grey</name>
-            <uri>file://media/materials/scripts/gazebo.material</uri>
-          </script>
-        </material>
-      </visual>
-      <self_collide>0</self_collide>
-      <enable_wind>0</enable_wind>
-      <kinematic>0</kinematic>
-    </link>
-  </model>
-  <joint name="connect_root_and_box" type="fixed">
-    <child link = "box_link"/>
-    <parent link = "world"/>
- </joint> -->
   <joint name="connect_root_and_world" type="fixed">
     <child link="root" />
     <parent link="world" />
-    <origin xyz="0.3 0.3 0.4" rpy="0 0 0" />
+    <origin xyz="0 0 0" rpy="0 0 0" />
   </joint>
   <xacro:property name="robot_root" value="root" />

File: src/kinova_with_d435/urdf/kinova_with_d435.xacro (robot description, xacro)
@@ -1,11 +1,14 @@
 <?xml version="1.0"?>
-<robot xmlns:xacro="http://www.ros.org/wiki/xacro" name="j2s7s300">
+<robot xmlns:xacro="http://www.ros.org/wiki/xacro" name="mrobot0_with_j2s7s300">
     <!-- include kinova arm -->
-    <xacro:include filename="$(find kinova_description)/urdf/j2s7s300_standalone.xacro"/>
+    <xacro:include filename="$(find kinova_description)/urdf/j2s7s300.xacro"/>
     <!-- include d435 camera -->
     <xacro:include filename="$(find realsense_ros_gazebo)/xacro/depthcam.xacro"/>
+    <!-- include mrobot0 -->
+    <xacro:include filename="$(find mrobot0)/urdf/mrobot0.urdf"/>
     <!-- add camera -->
     <xacro:realsense_d435 sensor_name="camera" parent_link="j2s7s300_link_7" rate="30.0">
-    <origin rpy="0 1.5707 0" xyz="0.06 0 -0.12"/>
+        <origin rpy="0 1.5707 0" xyz="0.06 0 -0.12"/>
     </xacro:realsense_d435>
+    <xacro:j2s7s300  base_parent="base_link"/>
 </robot>
