Commit message: change gpd cloud

File: src/kinova_with_d435/urdf/kinova_with_d435.xacro (robot description, xacro)
@@ -11,4 +11,10 @@
         <origin rpy="0 1.5707 0" xyz="0.06 0 -0.12"/>
     </xacro:realsense_d435>
+    <link name="root"/>
+    <joint name="connect_root_and_world" type="fixed">
+        <child link="root" />
+        <parent link="base_link" />
+        <origin xyz="0 0 0" rpy="0 0 0" />
+    </joint>
     <xacro:j2s7s300  base_parent="base_link"/>
 </robot>
